Commit message: Create launch file for Gazebo simulator.

File: urdf/material.xacro (robot description, xacro)
@@ -4,4 +4,10 @@
   <!-- Definitions of materials                 -->
   <!-- ======================================== -->
+  <material name="black">
+    <color rgba="0.0 0.0 0.0 1.0" />
+  </material>
+  <material name="white">
+    <color rgba="1.0 1.0 1.0 1.0" />
+  </material>
   <material name="gray">
     <color rgba="0.2 0.2 0.2 1.0" />

File: urdf/model.urdf (robot description, URDF)
Before this commit: robot triple_pendulum, 6 links, 5 joints
Links:
- link base_link: mass None -> 1.0; geometry visual box size=1.4 0.01 0.01
Joints:
- joint base_joint: origin xyz=0.0 0.0 0.0 rpy=0.0 0.0 0.0 -> xyz=0.0 0.0 1.5 rpy=0.0 0.0 0.0

File: urdf/model.urdf.xacro (robot description, xacro)
@@ -18,5 +18,5 @@
   <xacro:triple_pendulum
     parent="world">
-    <origin xyz="0.0 0.0 0.0" rpy="0.0 0.0 0.0" />
+    <origin xyz="0.0 0.0 1.5" rpy="0.0 0.0 0.0" />
   </xacro:triple_pendulum>
   <!-- ======================================== -->

File: urdf/triple_pendulum.xacro (robot description, xacro)
@@ -18,5 +18,25 @@
     <!-- ======================================== -->
     <!-- base_link -->
-    <link name="base_link" />
+    <link name="base_link">
+      <visual>
+        <origin xyz="0.0 0.0 0.0" rpy="0.0 0.0 0.0" />
+        <geometry>
+          <box size="1.4 0.01 0.01" />
+        </geometry>
+        <material name="black" />
+      </visual>
+      <!-- dummy -->
+      <inertial>
+        <origin xyz="0.0 0.0 0.0" rpy="0.0 0.0 0.0" />
+        <mass value="1.0" />
+        <inertia
+          ixx="0.01"
+          iyy="0.01"
+          izz="0.01"
+          ixy="0.0"
+          iyz="0.0"
+          ixz="0.0" />
+      </inertial>
+    </link>
     <!-- cart -->
     <link name="cart">
